Commit message: Update URDF for track calibration

File: robot_files/abb_irb_6700_track_irtb_6004/4_urdfs/abb_irbt6004_670_support/urdf/abb_irb6700_175_305_ibois.xacro (robot description, xacro)
@@ -6,5 +6,6 @@
       <parent link="world" />
       <child link = "rob1_axis" />
-      <origin xyz="0 0.0 0.0" rpy="0.0 0.0 3.14159265358979323846" />
+      <!--<origin xyz="0 0.0 0.0" rpy="0.0 0.0 3.14159265358979323846" />-->
+      <origin xyz="0 0.0 0.0" rpy="-0.00031264124506612164 -0.00031250271915146547 0.0004431808433690596" /> <!--Update for the base frame of the track -->
   </joint>
   <xacro:abb_irb6700_175_305_ibois prefix="rob1_" />

File: robot_files/abb_irb_6700_track_irtb_6004/4_urdfs/abb_irbt6004_670_support/urdf/abb_irbt6004_670.xacro (robot description, xacro)
@@ -8,5 +8,5 @@
       </inertial>
       <visual>
-        <origin xyz="-3.35 0.0 0.0" />
+        <origin xyz="3.35 0.0 0.0" />
         <geometry>
           <mesh filename="package://abb_irbt6004_670_support/meshes/abb_irbt6004_670/visual/axis.stl"/>
@@ -15,5 +15,5 @@
       </visual>
       <collision>
-        <origin xyz="-3.35 0.0 0.0"/>
+        <origin xyz="3.35 0.0 0.0"/>
         <geometry>
           <mesh filename="package://abb_irbt6004_670_support/meshes/abb_irbt6004_670/collision/axis.stl"/>
@@ -24,5 +24,5 @@
       <parent link="${prefix}axis"/>
       <child  link="${prefix}pedestal"/>
-      <origin xyz="0 0 0.05" rpy="0 0 3.14159265358979323846 "/> <!--track origin or translation from origin-->
+      <origin xyz="0 0 0.05" rpy="0 0 0"/> <!--track origin or translation from origin-->
       <axis   xyz="1 0 0"/>
       <limit lower="0" upper="6.700" effort="100000" velocity="2.618" />  <!--track limits or length-->

Commit message: update local repo

File: robot_files/abb_irb_6700_track_irtb_6004/4_urdfs/abb_irbt6004_670_support/urdf/abb_irb6700_175_305_ibois.xacro (robot description, xacro)
@@ -1,4 +1,4 @@
 <?xml version="1.0"?>
-<robot name="abb_irb6700_175_305_ibois" xmlns:xacro="http://ros.org/wiki/xacro">
+<robot name="aurora" xmlns:xacro="http://ros.org/wiki/xacro">
   <xacro:include filename="$(find abb_irbt6004_670_support)/urdf/abb_irb6700_175_305_ibois_macro.xacro"/>
   <link name="world" />

File: robot_files/abb_irb_6700_track_irtb_6004/4_urdfs/abb_irbt6004_670_support/urdf/abb_irb6700_175_305_ibois_macro.xacro (robot description, xacro)
@@ -2,5 +2,4 @@
 <robot xmlns:xacro="http://wiki.ros.org/xacro">
   <xacro:macro name="abb_irb6700_175_305_ibois" params="prefix" >
-  <!--<xacro:macro name="abb_irb6700_175_305_ibois" params="prefix prefix_notused" >-->
     <xacro:include filename="$(find abb_resources)/urdf/common_materials.xacro"/>
     <xacro:include filename="$(find abb_irb6700_support)/urdf/irb6700_175_305_macro.xacro"/>

File: robot_files/abb_irb_6700_track_irtb_6004_2x/4_urdfs/abb_irbt6004_670_support/urdf/abb_irb6700_175_305_ibois_tworobots.xacro (robot description, xacro)
@@ -1,4 +1,4 @@
 <?xml version="1.0"?>
-<robot name="abb_irb6700_175_305_ibois" xmlns:xacro="http://ros.org/wiki/xacro">
+<robot name="aurora_iris" xmlns:xacro="http://ros.org/wiki/xacro">
   <!--linking another xacro file of the robot without rail-->
   <xacro:include filename="$(find abb_irbt6004_670_support)/urdf/abb_irb6700_175_305_ibois_macro.xacro"/>
@@ -8,5 +8,5 @@
       <parent link="world" />
       <child link = "rob1_axis" />
-      <origin xyz="-3.35 -1.5 0.0" rpy="0.0 0.0 0.0" /> <!--translation of the track-->
+      <origin xyz="0.0 0.0 0.0" rpy="0.0006690539774448019 0.000669029972214783 0.00003588000859488913" /> <!--translation of the track-->
   </joint>
   <xacro:abb_irb6700_175_305_ibois prefix="rob1_" /> <!--robot with different base rotation-->
@@ -14,5 +14,5 @@
       <parent link="world" />
       <child link = "rob2_axis" />
-      <origin xyz="3.35 1.5 0.0" rpy="0.0 0.0 3.14159265358979323846" /> <!--translation of the track-->
+      <origin xyz="6.3145407114902 3.6055713818138 0.0019451920794" rpy="-0.0071789973774038915 -0.005247652228420866 -3.1404366692360592" /> <!--translation of the track-->
   </joint>
   <xacro:abb_irb6700_175_305_crcl prefix="rob2_" /> <!--robot with different base rotation-->
